File: cetus-RP2040-CPU.kicad_sch (KiCad schematic)
At the start: 36 parts, among them J1 Conn_01x03, J2 Conn_01x02, J3 Conn_01x02, J4 Conn_02x03_Odd_Even, U2 W25Q128JVS, U3 RP2040, Y1 ABLS-12.000MHZ-B4-T, Y2 X322516MLB4SI

Commit message: Remove spare components and break-off tab
Also, fix PCB DRC errors/warnings:

- Create a custom symbol for header to match footprint with missing pads

- Create footprints for flash and crystal which have 3D models
Parts:
- removed C16, C18: 27p, Capacitor_SMD:C_0402_1005Metric, symbol Device:C
- removed R6: 100, Resistor_SMD:R_0402_1005Metric, symbol Device:R
- removed R7: 1k, Resistor_SMD:R_0402_1005Metric, symbol Device:R
- removed Y1: ABLS-12.000MHZ-B4-T, RP2040_minimal:Crystal_SMD_HC49-US, symbol Device:Crystal
- JP2: symbol Connector_Generic:Conn_02x18_Odd_Even -> custom:Conn_02x18_Odd_Even_exc_pins15_17
- U2: footprint Package_SO:SOIC-8_5.23x5.23mm_P1.27mm -> custom:SOIC-8_5.23x5.23mm_P1.27mm+model
Connections:
- no-connect marks 33 -> 37

Commit message: Fix silkscreen crystal designation text size
Parts:
- Y2: footprint X322516MLB4SI:OSC_X322516MLB4SI -> OSC_X322516MLB4SI
Changed lines of the file:
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@@
       (effects (font (size 1.27 1.27)) (justify left))
     )
-    (property "Footprint" "X322516MLB4SI:OSC_X322516MLB4SI" (at 77.47 215.9 0)
+    (property "Footprint" "OSC_X322516MLB4SI" (at 77.47 215.9 0)
       (effects (font (size 1.27 1.27)) (justify bottom) hide)
     )
